File: Electronics/Open-JIP(KiCad)/Open-JIP(KiCad)_T3.6.kicad_pcb (KiCad board)
At the start: 2 copper layers, 7.3 x 7.1 mm, 31 parts, among them J1 DCJ200-10-A-XX-X_REVA, J2 Screw_Terminal_01x02, U1 74HC4066D,653, U2 74HC4066D,653, U3 KA7812ETU, U4 OPA320AIDBVT, U5 Teensy3.6

Commit message: finalised v0.3 for teensy 3.6
Parts:
- added G***: LOGO, Silkscreen_Images:Open-JIP_Logo, F.Cu at (136.1, 106.2)
- added REF**: MountingHole_3.2mm_M3_ISO7380_Pad, MountingHole:MountingHole_3.2mm_M3_ISO7380_Pad, F.Cu at (184.9, 82.0)
- added REF**: MountingHole_3.2mm_M3_ISO7380_Pad, MountingHole:MountingHole_3.2mm_M3_ISO7380_Pad, F.Cu at (135.4, 82.0)
- J1: value DCJ200-10-A-XX-X_REVA -> EJ503A; footprint Additional-parts:GCT_DCJ200-10-A-XX-X_REVA -> Additional-parts:DCJack_MPD_EJ503A
- moved J1 3.82 mm to (181.1, 100.3)
- moved D1 0.10 mm to (148.5, 82.0)
- turned C4 to 270 degrees
Connections:
- U5 pad 32: ActinicGain1 -> Net-(U5-Pad32)
- U5 pad 33: ActinicGain2 -> Net-(U5-Pad33)
- U5 pad 34: ActinicGain3 -> Net-(U5-Pad34)
- U5 pad 35: ActinicGain4 -> Net-(U5-Pad35)
- U5 pad 37: Net-(U5-Pad37) -> ActinicGain3
- U5 pad 38: Net-(U5-Pad38) -> ActinicGain2
- U5 pad 43: Net-(U5-Pad43) -> ActinicGain1
- U5 pad 44: Net-(U5-Pad44) -> ActinicGain4
Routing:
- net +3V3: track 5.63 -> 88.0 mm, vias 0 -> 3
- net ActinicGain3: track 0.00 -> 16.0 mm, vias 0 -> 1
- net Net-(R6-Pad2): track 0.00 -> 14.7 mm, vias 0 -> 2
- net Net-(R4-Pad2): track 0.00 -> 13.9 mm
- net ActinicGain2: track 0.00 -> 13.7 mm, vias 0 -> 1
- net /TrigOut: track 0.00 -> 12.3 mm
- net ActinicGain4: track 0.00 -> 7.97 mm
- net Net-(R11-Pad2): track 0.00 -> 6.78 mm
- net ActinicGain1: track 0.00 -> 6.68 mm
- net Net-(R9-Pad2): track 0.00 -> 6.43 mm
- net GND: track 0.00 -> 5.31 mm, vias 0 -> 22
- net GNDA: track 0.00 -> 3.68 mm, vias 0 -> 26
- net /Out: track 23.1 -> 20.2 mm
- net /-IN: track 62.2 -> 61.3 mm, vias 4 -> 5
- net (no net): vias 0 -> 2
- added copper zone on F.Cu, net +15V
- added copper zone on B.Cu, net GND
- added copper zone on F.Cu, net GND
- added copper zone on B.Cu, net GNDA
- added copper zone on F.Cu, net GNDA
- added copper zone on F.Cu, net Net-(C4-Pad2)
- added copper zone on B.Cu, net Net-(C7-Pad2)
- added copper zone on F.Cu, net Net-(C7-Pad2)
Other:
- board size 7.3 x 7.1 mm -> 61.7 x 35.3 mm
- board text added: "+"
- board text added: "-"
- board text added: "Bates et al. 2019"
- board text added: "v0.3"
