File: Electronics/Open-JIP(KiCad)/Open-JIP(KiCad)_T3.2/Open-JIP(KiCad)_T3.2.kicad_pcb (KiCad board)
At the start: 2 copper layers, 31 parts, among them J1 EJ503A, J2 Screw_Terminal_01x02, U1 74HC4066D,653, U2 KA7812ETU, U3 74HC4066D,653, U4 OPA320AIDBVT, U5 Teensy3.2

Commit message: finished v0.3 for teensy 3.2 and added gerber files
Parts:
- removed D2: LED, LED_SMD:LED_0805_2012Metric_Pad1.15x1.40mm_HandSolder
- removed R12: 1K, Resistor_SMD:R_0805_2012Metric_Pad1.20x1.40mm_HandSolder
- added REF**: MountingHole_3.2mm_M3_DIN965_Pad, MountingHole:MountingHole_3.2mm_M3_DIN965_Pad, F.Cu at (120.0, 76.7)
- added REF**: MountingHole_3.2mm_M3_DIN965_Pad, MountingHole:MountingHole_3.2mm_M3_DIN965_Pad, F.Cu at (120.0, 30.0)
- moved U2 61.7 mm to (119.1, 38.6)
- moved C4 61.2 mm to (113.0, 34.8), turned to 0 degrees
- moved C2 60.7 mm to (120.4, 34.8), turned to 0 degrees
- moved J1 59.7 mm to (127.5, 39.4)
- moved C6 59.7 mm to (106.7, 39.4)
- moved R13 51.8 mm to (121.4, 43.7), turned to 180 degrees
- moved D3 50.0 mm to (117.3, 43.7), turned to 0 degrees
- moved J2 39.9 mm to (108.7, 46.0)
- moved U1 38.4 mm to (132.6, 49.3)
- moved R10 38.1 mm to (123.2, 52.8)
- moved R3 38.1 mm to (123.2, 46.0)
- moved R5 38.1 mm to (123.2, 48.3)
- moved R7 38.1 mm to (123.2, 50.5)
- moved CR1 37.9 mm to (119.1, 46.7)
- moved D1 9.23 mm to (109.0, 64.0)
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Connections:
- C5 pad 2: Net-(C5-Pad2) -> GNDA
- U4 pad 2: Net-(C5-Pad2) -> GNDA
- U5 pad 17: GND -> Net-(U5-Pad17)
- U5 pad 27: ActinicGain4 -> FluoroGain3
- U5 pad 28: ActinicGain3 -> FluoroGain2
- U5 pad 29: ActinicGain1 -> FluoroGain4
- U5 pad 30: ActinicGain2 -> FluoroGain1
- U5 pad 5: FluoroGain1 -> ActinicGain1
- U5 pad 6: FluoroGain2 -> ActinicGain4
- U5 pad 7: FluoroGain3 -> ActinicGain2
- U5 pad 8: FluoroGain4 -> ActinicGain3
Routing:
- net +5V: track 13.6 -> 0.00 mm
- net ActinicGain1: track 23.9 -> 11.4 mm, vias 1 -> 0
- net ActinicGain4: track 24.7 -> 12.9 mm, vias 1 -> 0
- net ActinicGain2: track 5.42 -> 16.9 mm, vias 0 -> 1
- net FluoroGain1: track 18.3 -> 7.53 mm
- net FluoroGain4: track 19.5 -> 9.14 mm, vias 2 -> 0
- net +3V3: track 61.1 -> 70.9 mm, vias 1 -> 2
- net ActinicGain3: track 9.02 -> 18.3 mm, vias 0 -> 1
- net GNDA: track 0.00 -> 7.94 mm, vias 0 -> 24
- net FluoroGain2: track 8.65 -> 14.0 mm
- net Net-(C5-Pad2): track 4.55 -> 0.00 mm
- net Net-(C1-Pad2): track 9.50 -> 14.0 mm
- net FluoroGain3: track 9.81 -> 14.1 mm
- net Net-(R10-Pad2): track 14.1 -> 17.6 mm
- net Net-(R7-Pad2): track 11.9 -> 14.6 mm
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- added copper zone on B.Cu, net GND
- added copper zone on F.Cu, net GND
- added copper zone on B.Cu, net GNDA
- added copper zone on F.Cu, net GNDA
Other:
- board outline added: 36.2 x 53.7 mm
- board text added: "+"
- board text added: "-"
