File: Electronics/Open-JIP(KiCad)/Open-JIP(KiCad)_T3.2/Open-JIP(KiCad)_T3.2.sch (KiCad schematic (older format))
At the start: 31 parts, among them J1 EJ503A, J2 Screw_Terminal_01x02, U1 74HC4066D,653, U2 KA7812ETU, U3 74HC4066D,653, U4 OPA320AIDBVT, U5 Teensy3.2

Commit message: finished v0.3 for teensy 3.2 and added gerber files
Parts:
- removed D2: LED, LED_SMD:LED_0805_2012Metric_Pad1.15x1.40mm_HandSolder, symbol Device:LED
- removed R12: 1K, Resistor_SMD:R_0805_2012Metric_Pad1.20x1.40mm_HandSolder, symbol Device:R
Connections:
- net ActinicGain1: now also U5.5 (3_TX_PWM); no longer U5.29 (22_A8_Touch_PWM)
- net ActinicGain2: now also U5.7 (5_TX1_PWM); no longer U5.30 (23_A9_Touch_PWM)
- net ActinicGain3: now also U5.8 (6_PWM); no longer U5.28 (21_A7_RX1_CS_PWM)
- net ActinicGain4: now also U5.6 (4_RX_PWM); no longer U5.27 (20_A6_CS_PWM)
- net FluoroGain1: now also U5.30 (23_A9_Touch_PWM); no longer U5.5 (3_TX_PWM)
- net FluoroGain2: now also U5.28 (21_A7_RX1_CS_PWM); no longer U5.6 (4_RX_PWM)
- net FluoroGain3: now also U5.27 (20_A6_CS_PWM); no longer U5.7 (5_TX1_PWM)
- net FluoroGain4: now also U5.29 (22_A8_Touch_PWM); no longer U5.8 (6_PWM)
- net GND: no longer U5.17 (GND)
- net GNDA: now also C5.2, U4.2 (V-)
Changed lines of the file:
@@
 Connection ~ 4650 3450
-Wire Wire Line
-	4500 3850 4650 3850
 Wire Wire Line
 	4500 3250 4850 3250
@@
 Wire Wire Line
 	1900 5150 1900 5300
+Text GLabel 7800 1650 0    50   Input ~ 0
+ActinicGain1
+Text GLabel 7800 1850 0    50   Input ~ 0
+ActinicGain2
+Text GLabel 7800 1950 0    50   Input ~ 0
+ActinicGain3
+Text GLabel 7800 1750 0    50   Input ~ 0
+ActinicGain4
+Text GLabel 9800 3850 2    50   Input ~ 0
+FluoroGain1
+Text GLabel 7800 3950 0    50   Input ~ 0
+FluoroGain2
+Text GLabel 7800 3850 0    50   Input ~ 0
+FluoroGain3
 Text GLabel 9800 3950 2    50   Input ~ 0
-ActinicGain1
-Text GLabel 9800 3850 2    50   Input ~ 0
-ActinicGain2
-Text GLabel 7800 3950 0    50   Input ~ 0
-ActinicGain3
-Text GLabel 7800 3850 0    50   Input ~ 0
-ActinicGain4
-Text GLabel 7800 1650 0    50   Input ~ 0
-FluoroGain1
-Text GLabel 7800 1750 0    50   Input ~ 0
-FluoroGain2
-Text GLabel 7800 1850 0    50   Input ~ 0
-FluoroGain3
-Text GLabel 7800 1950 0    50   Input ~ 0
 FluoroGain4
 $Comp
@@
 $EndComp
 $Comp
-L power:GND #PWR0118
-U 1 1 5FE91B90
-P 7800 2850
-F 0 "#PWR0118" H 7800 2600 50  0001 C CNN
-F 1 "GND" V 7805 2722 50  0000 R CNN
-F 2 "" H 7800 2850 50  0001 C CNN
-F 3 "" H 7800 2850 50  0001 C CNN
-	1    7800 2850
-	0    1    1    0
-$EndComp
-$Comp
-L Device:R R12
-U 1 1 5FE92923
-P 7250 5350
-F 0 "R12" H 7320 5396 50  0000 L CNN
-F 1 "1K" H 7320 5305 50  0000 L CNN
-F 2 "Resistor_SMD:R_0805_2012Metric_Pad1.20x1.40mm_HandSolder" V 7180 5350 50  0001 C CNN
-F 3 "~" H 7250 5350 50  0001 C CNN
-	1    7250 5350
-	1    0    0    -1
-$EndComp
-$Comp
 L Device:R R13
 U 1 1 5FE92BE8
@@
 	4500 5150 4850 5150
 $Comp
-L power:+5V #PWR0121
-U 1 1 5FE93F51
-P 7250 5100
-F 0 "#PWR0121" H 7250 4950 50  0001 C CNN
-F 1 "+5V" H 7265 5273 50  0000 C CNN
-F 2 "" H 7250 5100 50  0001 C CNN
-F 3 "" H 7250 5100 50  0001 C CNN
-	1    7250 5100
-	1    0    0    -1
-$EndComp
-$Comp
 L power:+15V #PWR0122
 U 1 1 5FE946B7
@@
 	1    7750 5100
 	1    0    0    -1
-$EndComp
-$Comp
-L Device:LED D2
-U 1 1 5FE957E5
-P 7250 5750
-F 0 "D2" V 7289 5632 50  0000 R CNN
-F 1 "LED" V 7198 5632 50  0000 R CNN
-F 2 "LED_SMD:LED_0805_2012Metric_Pad1.15x1.40mm_HandSolder" H 7250 5750 50  0001 C CNN
-F 3 "~" H 7250 5750 50  0001 C CNN
-	1    7250 5750
-	0    -1   -1   0
 $EndComp
 $Comp
@@
 $EndComp
 $Comp
-L power:GND #PWR0123
-U 1 1 5FE96F8E
-P 7250 6000
-F 0 "#PWR0123" H 7250 5750 50  0001 C CNN
-F 1 "GND" H 7255 5827 50  0000 C CNN
-F 2 "" H 7250 6000 50  0001 C CNN
-F 3 "" H 7250 6000 50  0001 C CNN
-	1    7250 6000
-	1    0    0    -1
-$EndComp
-$Comp
 L power:GND #PWR0124
 U 1 1 5FE974D6
@@
 $EndComp
 Wire Wire Line
-	7250 6000 7250 5900
-Wire Wire Line
-	7250 5600 7250 5500
-Wire Wire Line
 	7750 5600 7750 5500
 Wire Wire Line
@@
 Wire Wire Line
 	7750 5200 7750 5100
-Wire Wire Line
-	7250 5200 7250 5100
 Wire Notes Line
 	1100 750  6350 750
@@
 Text GLabel 7800 3550 0    50   Input ~ 0
 FluoroRead
+Wire Wire Line
+	4550 4150 4650 4150
+Wire Wire Line
+	4500 3850 4550 3850
+Wire Wire Line
+	4550 3850 4550 4150
+Connection ~ 4550 3850
+Wire Wire Line
+	4550 3850 4650 3850
+Connection ~ 4650 4150
 $EndSCHEMATC
