File: electronics/v0.3/open_jip/open_jip.kicad_pcb (KiCad board)
At the start: 2 copper layers, 61.7 x 35.3 mm, 25 parts, among them J1 EJ503A, J2 Screw_Terminal_01x02, U1 KA7812ETU, U2 OPA320AIDBVT, U3 Teensy3.6

Commit message: rename file structure for v0.3
Parts:
- G***: footprint Silkscreen_Images:Open-JIP_Logo -> Silkscreen_Images:open_jip_Logo
Changed lines of the file:
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@@
     (descr "LED SMD 0805 (2012 Metric), square (rectangular) end terminal, IPC_7351 nominal, (Body size source: https://docs.google.com/spreadsheets/d/1BsfQQcO9C6DZCsRaXUlFlo91Tg2WpOkGARC1WS5S8t0/edit?usp=sharing), generated with kicad-footprint-generator")
     (tags "LED handsolder")
-    (property "Sheetfile" "Open-JIP.kicad_sch")
+    (property "Sheetfile" "open_jip.kicad_sch")
     (property "Sheetname" "")
     (attr smd)
@@
     (descr "Resistor SMD 0805 (2012 Metric), square (rectangular) end terminal, IPC_7351 nominal with elongated pad for handsoldering. (Body size source: IPC-SM-782 page 72, https://www.pcb-3d.com/wordpress/wp-content/uploads/ipc-sm-782a_amendment_1_and_2.pdf), generated with kicad-footprint-generator")
     (tags "resistor handsolder")
-    (property "Sheetfile" "Open-JIP.kicad_sch")
+    (property "Sheetfile" "open_jip.kicad_sch")
     (property "Sheetname" "")
     (attr smd)
@@
     (descr "Capacitor SMD 0805 (2012 Metric), square (rectangular) end terminal, IPC_7351 nominal with elongated pad for handsoldering. (Body size source: IPC-SM-782 page 76, https://www.pcb-3d.com/wordpress/wp-content/uploads/ipc-sm-782a_amendment_1_and_2.pdf, https://docs.google.com/spreadsheets/d/1BsfQQcO9C6DZCsRaXUlFlo91Tg2WpOkGARC1WS5S8t0/edit?usp=sharing), generated with kicad-footprint-generator")
     (tags "capacitor handsolder")
-    (property "Sheetfile" "Open-JIP.kicad_sch")
+    (property "Sheetfile" "open_jip.kicad_sch")
     (property "Sheetname" "")
     (attr smd)
@@
     (descr "Capacitor SMD 0805 (2012 Metric), square (rectangular) end terminal, IPC_7351 nominal with elongated pad for handsoldering. (Body size source: IPC-SM-782 page 76, https://www.pcb-3d.com/wordpress/wp-content/uploads/ipc-sm-782a_amendment_1_and_2.pdf, https://docs.google.com/spreadsheets/d/1BsfQQcO9C6DZCsRaXUlFlo91Tg2WpOkGARC1WS5S8t0/edit?usp=sharing), generated with kicad-footprint-generator")
     (tags "capacitor handsolder")
-    (property "Sheetfile" "Open-JIP.kicad_sch")
+    (property "Sheetfile" "open_jip.kicad_sch")
     (property "Sheetname" "")
     (attr smd)
@@
     (descr "SMD capacitor, aluminum electrolytic, Panasonic A5 / Nichicon, 4.0x5.4mm")
     (tags "capacitor electrolytic")
-    (property "Sheetfile" "Open-JIP.kicad_sch")
+    (property "Sheetfile" "open_jip.kicad_sch")
     (property "Sheetname" "")
     (attr smd)
@@
   (footprint "Additional-parts:BD681" (layer "F.Cu")
     (at 147.549 101.2)
-    (property "Sheetfile" "Open-JIP.kicad_sch")
+    (property "Sheetfile" "open_jip.kicad_sch")
     (property "Sheetname" "")
     (attr through_hole)
@@
     (property "PARTREV" "1.3")
     (property "STANDARD" "Manufacturer Recommendations")
-    (property "Sheetfile" "Open-JIP.kicad_sch")
+    (property "Sheetfile" "open_jip.kicad_sch")
     (property "Sheetname" "")
     (attr through_hole)
@@
     (descr "Altech AK300 terminal block, pitch 5.0mm, 45 degree angled, see http://www.mouser.com/ds/2/16/PCBMETRC-24178.pdf")
     (tags "Altech AK300 terminal block pitch 5.0mm")
-    (property "Sheetfile" "Open-JIP.kicad_sch")
+    (property "Sheetfile" "open_jip.kicad_sch")
     (property "Sheetname" "")
     (attr through_hole)
@@
     (property "Manufacturer" "ON Semiconductor")
     (property "Package" "TO253P1067X470X2040-3")
-    (property "Sheetfile" "Open-JIP.kicad_sch")
+    (property "Sheetfile" "open_jip.kicad_sch")
     (property "Sheetname" "")
     (attr through_hole)
@@
   (footprint "Additional-parts:SOT95P280X145-5N" (layer "F.Cu")
     (at 161.4 81.9)
-    (property "Sheetfile" "Open-JIP.kicad_sch")
+    (property "Sheetfile" "open_jip.kicad_sch")
     (property "Sheetname" "")
     (attr through_hole)
@@
   (footprint "Teensy:Teensy35_36" (layer "F.Cu")
     (at 160.225001 82.265001 180)
-    (property "Sheetfile" "Open-JIP.kicad_sch")
+    (property "Sheetfile" "open_jip.kicad_sch")
     (property "Sheetname" "")
     (attr through_hole)
@@
     (property "PARTREV" "B")
     (property "STANDARD" "Manufacturer Recommendations")
-    (property "Sheetfile" "Open-JIP.kicad_sch")
+    (property "Sheetfile" "open_jip.kicad_sch")
     (property "Sheetname" "")
     (attr through_hole)
@@
     (pad "1" thru_hole circle locked (at 0 0) (size 5.7 5.7) (drill 3.2) (layers *.Cu *.Mask))
   )
-  (footprint "Silkscreen_Images:Open-JIP_Logo" (layer "F.Cu")
+  (footprint "Silkscreen_Images:open_jip_Logo" (layer "F.Cu")
     (at 142.828 82.394 -90)
     (attr through_hole)
@@
     (descr "Capacitor SMD 0805 (2012 Metric), square (rectangular) end terminal, IPC_7351 nominal with elongated pad for handsoldering. (Body size source: IPC-SM-782 page 76, https://www.pcb-3d.com/wordpress/wp-content/uploads/ipc-sm-782a_amendment_1_and_2.pdf, https://docs.google.com/spreadsheets/d/1BsfQQcO9C6DZCsRaXUlFlo91Tg2WpOkGARC1WS5S8t0/edit?usp=sharing), generated with kicad-footprint-generator")
     (tags "capacitor handsolder")
-    (property "Sheetfile" "Open-JIP.kicad_sch")
+    (property "Sheetfile" "open_jip.kicad_sch")
     (property "Sheetname" "")
     (attr smd)
@@
     (descr "Resistor SMD 0805 (2012 Metric), square (rectangular) end terminal, IPC_7351 nominal with elongated pad for handsoldering. (Body size source: IPC-SM-782 page 72, https://www.pcb-3d.com/wordpress/wp-content/uploads/ipc-sm-782a_amendment_1_and_2.pdf), generated with kicad-footprint-generator")
     (tags "resistor handsolder")
-    (property "Sheetfile" "Open-JIP.kicad_sch")
+    (property "Sheetfile" "open_jip.kicad_sch")
     (property "Sheetname" "")
     (attr smd)
@@
     (descr "Resistor SMD 0805 (2012 Metric), square (rectangular) end terminal, IPC_7351 nominal with elongated pad for handsoldering. (Body size source: IPC-SM-782 page 72, https://www.pcb-3d.com/wordpress/wp-content/uploads/ipc-sm-782a_amendment_1_and_2.pdf), generated with kicad-footprint-generator")
     (tags "resistor handsolder")
-    (property "Sheetfile" "Open-JIP.kicad_sch")
+    (property "Sheetfile" "open_jip.kicad_sch")
     (property "Sheetname" "")
     (attr smd)
@@
     (descr "Capacitor SMD 0805 (2012 Metric), square (rectangular) end terminal, IPC_7351 nominal with elongated pad for handsoldering. (Body size source: IPC-SM-782 page 76, https://www.pcb-3d.com/wordpress/wp-content/uploads/ipc-sm-782a_amendment_1_and_2.pdf, https://docs.google.com/spreadsheets/d/1BsfQQcO9C6DZCsRaXUlFlo91Tg2WpOkGARC1WS5S8t0/edit?usp=sharing), generated with kicad-footprint-generator")
     (tags "capacitor handsolder")
-    (property "Sheetfile" "Open-JIP.kicad_sch")
+    (property "Sheetfile" "open_jip.kicad_sch")
     (property "Sheetname" "")
     (attr smd)
@@
   (footprint "35602R2JT:35602R2JT" (layer "F.Cu")
     (at 149.9556 95.3)
-    (property "Sheetfile" "Open-JIP.kicad_sch")
+    (property "Sheetfile" "open_jip.kicad_sch")
     (property "Sheetname" "")
     (attr through_hole)
@@
     (descr "Resistor SMD 0805 (2012 Metric), square (rectangular) end terminal, IPC_7351 nominal with elongated pad for handsoldering. (Body size source: IPC-SM-782 page 72, https://www.pcb-3d.com/wordpress/wp-content/uploads/ipc-sm-782a_amendment_1_and_2.pdf), generated with kicad-footprint-generator")
     (tags "resistor handsolder")
-    (property "Sheetfile" "Open-JIP.kicad_sch")
+    (property "Sheetfile" "open_jip.kicad_sch")
     (property "Sheetname" "")
     (attr smd)
@@
     (descr "Capacitor SMD 0805 (2012 Metric), square (rectangular) end terminal, IPC_7351 nominal with elongated pad for handsoldering. (Body size source: IPC-SM-782 page 76, https://www.pcb-3d.com/wordpress/wp-content/uploads/ipc-sm-782a_amendment_1_and_2.pdf, https://docs.google.com/spreadsheets/d/1BsfQQcO9C6DZCsRaXUlFlo91Tg2WpOkGARC1WS5S8t0/edit?usp=sharing), generated with kicad-footprint-generator")
     (tags "capacitor handsolder")
-    (property "Sheetfile" "Open-JIP.kicad_sch")
+    (property "Sheetfile" "open_jip.kicad_sch")
     (property "Sheetname" "")
     (attr smd)
@@
   (footprint "3386G-1-102LF:3386G-1-102LF" (layer "F.Cu")
     (at 169.0482 99.1618 -90)
-    (property "Sheetfile" "Open-JIP.kicad_sch")
+    (property "Sheetfile" "open_jip.kicad_sch")
     (property "Sheetname" "")
     (attr through_hole)
@@
     (descr "Resistor SMD 0805 (2012 Metric), square (rectangular) end terminal, IPC_7351 nominal with elongated pad for handsoldering. (Body size source: IPC-SM-782 page 72, https://www.pcb-3d.com/wordpress/wp-content/uploads/ipc-sm-782a_amendment_1_and_2.pdf), generated with kicad-footprint-generator")
     (tags "resistor handsolder")
-    (property "Sheetfile" "Open-JIP.kicad_sch")
+    (property "Sheetfile" "open_jip.kicad_sch")
     (property "Sheetname" "")
     (attr smd)
@@
     (descr "Capacitor SMD 0805 (2012 Metric), square (rectangular) end terminal, IPC_7351 nominal with elongated pad for handsoldering. (Body size source: IPC-SM-782 page 76, https://www.pcb-3d.com/wordpress/wp-content/uploads/ipc-sm-782a_amendment_1_and_2.pdf, https://docs.google.com/spreadsheets/d/1BsfQQcO9C6DZCsRaXUlFlo91Tg2WpOkGARC1WS5S8t0/edit?usp=sharing), generated with kicad-footprint-generator")
     (tags "capacitor handsolder")
-    (property "Sheetfile" "Open-JIP.kicad_sch")
+    (property "Sheetfile" "open_jip.kicad_sch")
     (property "Sheetname" "")
     (attr smd)
