File: electronics/open-jip/flu_detect.kicad_sch (KiCad schematic)
At the start: 8 parts

Commit message: updating PCB layout
Parts:
- U?: footprint op_amps:OPA328DBVR -> Package_TO_SOT_SMD:SOT-23-6
Changed lines of the file:
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@@
       (effects (font (size 1.524 1.524)))
     )
-    (property "Footprint" "op_amps:OPA328DBVR" (at 134.62 104.14 0)
+    (property "Footprint" "Package_TO_SOT_SMD:SOT-23-6" (at 134.62 104.14 0)
       (effects (font (size 1.27 1.27) italic) hide)
     )
