File: electronics/open-jip/open-jip.kicad_pcb (KiCad board)
At the start: 2 copper layers, 50 parts, among them J1 Conn_01x05_Socket, J2 TBP02R2-381-02BE, J3 PJ-002A, J4 TBP02R2-381-02BE, J5 Conn_ARM_JTAG_SWD_10, J6 Conn_01x05_Socket, Q1 DMP6023LE-13, U1 STM32L432KCU6, U2 AP63205WU-7, U3 ADP122AUJZ-3.3-R7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

Commit message: updating PCB layout
Parts:
- D2: moved to B.Cu
- U4: footprint op_amps:OPA328DBVR -> Package_TO_SOT_SMD:SOT-23-6
- moved CR1 104.1 mm to (194.0, 59.2), turned to -90 degrees
- moved F2 101.3 mm to (201.4, 72.3)
- moved J4 98.5 mm to (203.2, 64.4), turned to 180 degrees
- moved U5 83.3 mm to (190.0, 75.1), turned to 90 degrees
- moved R8 81.8 mm to (190.8, 60.2), turned to 90 degrees
- moved C18 79.9 mm to (200.7, 78.2)
- moved R7 78.2 mm to (190.8, 63.7), turned to 90 degrees
- moved R4 74.6 mm to (180.6, 54.6), turned to 90 degrees
- moved R6 70.0 mm to (170.5, 58.7), turned to 90 degrees
- moved R3 69.7 mm to (180.6, 58.2), turned to 90 degrees
- moved R5 68.6 mm to (175.9, 61.4)
- moved U4 68.0 mm to (176.0, 58.5), turned to 180 degrees
- moved C16 68.0 mm to (175.9, 63.5)
- moved C17 66.6 mm to (189.9, 86.6)
- moved C15 66.1 mm to (172.7, 60.6), turned to -90 degrees
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Routing:
- net NRST: track 0.00 -> 46.1 mm, vias 0 -> 2
- net /TRST_PB4: track 0.00 -> 28.3 mm
- net /TDI_PA15: track 0.00 -> 21.7 mm
- net /PA7: track 0.00 -> 21.2 mm, vias 0 -> 2
- net /TDO/SWO_PB3: track 0.00 -> 19.9 mm
- net /PA6: track 0.00 -> 17.9 mm
- net /TMS/SWDAT_PA13: track 0.00 -> 17.8 mm
- net /TCK/SWCLK_PA14: track 0.00 -> 17.5 mm
- net +3.3V: track 0.00 -> 16.0 mm, vias 0 -> 2
- net +5V: track 0.00 -> 15.6 mm, vias 0 -> 2
- net Net-(D2-K): track 0.00 -> 11.0 mm
- net /ADC1_IN5: track 0.00 -> 9.83 mm
- net Net-(U1-PC15): track 0.00 -> 9.02 mm
- net /USART1_TX: track 0.00 -> 6.81 mm
- net Net-(U1-PC14): track 0.00 -> 6.66 mm
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- added copper zone on F.Cu, net +5V
- added copper zone on B.Cu, net GND
- added copper zone on F.Cu, net GND
- added copper zone on F.Cu, net Net-(U2-SW)
Other:
- board outline added: 47.1 x 54.5 mm
