File: electronics/detect/detect.kicad_pcb (KiCad board)
At the start: 2 copper layers, 29.1 x 45.1 mm, 29 parts, among them J1 Conn_02x06_Counter_Clockwise, J2 Conn_01x04_Socket, J3 Conn_ARM_JTAG_SWD_10, U1 STM32L432KCU6, U2 OPA328DBVR, Y1 ECS-.327-12.5-34R-C-TR

Commit message: working on cuvette mount and finished routing both pcbs
Parts:
- added REF**: MountingHole_3.2mm_M3, MountingHole:MountingHole_3.2mm_M3, F.Cu at (193.0, 62.5)
Routing:
- net GND: track 4.92 -> 20.9 mm, vias 14 -> 28
- net /TRST_PB4: track 13.8 -> 19.1 mm
- net Net-(J3-GNDDetect): track 0.04 -> 2.80 mm
- net /PA6: track 29.7 -> 28.1 mm
- net +3.3V: track 90.5 -> 89.4 mm
- net /USART1_TX: track 5.71 -> 4.78 mm
